Commit message: Add simple URDF of SeekurJr

File: examples/seekurjr.urdf (robot description, URDF)
Before this commit: robot seekurjr, 2 links, 1 joints
Links:
- added link velodyne
Joints:
- removed joint offset
- added joint lower_dynamixel: type fixed, parent body, child lower_dynamixel, origin xyz=0 0 0.05 rpy=0 0 0
- added joint velodyne: type fixed, parent body, child velodyne, origin xyz=0.3 0.22 0.45 rpy=0 0 0

Commit message: fixed cdff_envire.load_urdf

File: examples/seekurjr.urdf (robot description, URDF)
Before this commit: robot seekurjr, 3 links, 2 joints
Links:
- link body: geometry visual sphere radius=0.5
